Commit message: fix: PhysX phantom mass, combined force call, world-frame target position
- quad.urdf: arm_motor_* mass 0→0.001 kg, inertia 0→1e-6 diagonal
  PhysX was adding ~1.1 kg phantom mass per link with mass=0+inertia=0
  (total 4.5 kg phantom vs 0.25 kg intended), causing drone to free-fall
- aerial_gym_base_env: combine drag+motor forces into single
  set_external_force_and_torque call — second call with all-zero drag was
  setting has_external_wrench=False and silently disabling motor thrust
- position_setpoint_env: target_position = env_origins + offset
  In Isaac Lab all envs share world space; target=(0,0,0) gave 219m initial
  dist with 1024 envs, immediately triggering crash condition

Co-Authored-By: Claude Sonnet 4.6 <noreply@anthropic.com>

File: resources/robots/quad/quad.urdf (robot description, URDF)
Before this commit: robot quadrotor, 9 links, 8 joints
Links:
- link arm_motor_0: mass 0.0 -> 0.001
- link arm_motor_1: mass 0.0 -> 0.001
- link arm_motor_2: mass 0.0 -> 0.001
- link arm_motor_3: mass 0.0 -> 0.001
